Commit message: using unique usb address

File: open_manipulator_description/ros2_control/omy_l100_current.ros2_control.xacro (robot description, xacro)
@@ -1,5 +1,5 @@
 <?xml version="1.0"?>
 <robot xmlns:xacro="http://www.ros.org/wiki/xacro">
-  <xacro:macro name="omy_l100_system" params="name prefix port_name:=^|/dev/ttyUSB0 use_sim:=^|false use_mock_hardware:=^|false mock_sensor_commands:=^|false">
+  <xacro:macro name="omy_l100_system" params="name prefix port_name:=^|/dev/serial/by-id/usb-FTDI_USB__-__Serial_Converter_FTAK89CW-if00-port0 use_sim:=^|false use_mock_hardware:=^|false mock_sensor_commands:=^|false">
     <ros2_control name="${name}" type="system">
       <xacro:if value="$(arg use_sim)">

File: open_manipulator_description/ros2_control/omy_l100_position.ros2_control.xacro (robot description, xacro)
@@ -1,5 +1,5 @@
 <?xml version="1.0"?>
 <robot xmlns:xacro="http://www.ros.org/wiki/xacro">
-  <xacro:macro name="omy_l100_system" params="name prefix port_name:=^|/dev/ttyUSB0 use_sim:=^|false use_mock_hardware:=^|false mock_sensor_commands:=^|false">
+  <xacro:macro name="omy_l100_system" params="name prefix port_name:=^|/dev/serial/by-id/usb-FTDI_USB__-__Serial_Converter_FTAK89CW-if00-port0 use_sim:=^|false use_mock_hardware:=^|false mock_sensor_commands:=^|false">
     <ros2_control name="${name}" type="system">
       <xacro:if value="$(arg use_sim)">
@@ -17,5 +17,4 @@
           <xacro:unless value="${use_mock_hardware}">
             <plugin>dynamixel_hardware_interface/DynamixelHardware</plugin>
-            <param name="port_name">${port_name}</paramport_name:=^|/dev/serial/by-id/usb-FTDI_USB__-__Serial_Converter_FTAK89CW-if00-port0>
             <param name="port_name">${port_name}</param>
             <param name="baud_rate">4000000</param>

File: open_manipulator_description/urdf/omy_l100/omy_l100.urdf.xacro (robot description, xacro)
@@ -5,5 +5,5 @@
   <xacro:arg name="use_mock_hardware" default="false" />
   <xacro:arg name="mock_sensor_commands" default="false" />
-  <xacro:arg name="port_name" default="/dev/ttyUSB0" />
+  <xacro:arg name="port_name" default="/dev/serial/by-id/usb-FTDI_USB__-__Serial_Converter_FTAK89CW-if00-port0" />
   <xacro:arg name="ros2_control_type" default="omy_l100_current" />
   <xacro:include filename="$(find open_manipulator_description)/urdf/omy_l100/omy_l100_arm.urdf.xacro" />
