Commit message: Add fixed OMY teleop task frame
Co-authored-by: Soomi Lee <soomi_lee@berkeley.edu>

File: open_manipulator_description/urdf/omy_l100/omy_l100.urdf.xacro (robot description, xacro)
@@ -17,4 +17,12 @@
   </joint>
   <xacro:omy_l100 prefix="$(arg prefix)" />
+  <!-- Fixed teleoperation endpoint at the gripper-joint origin. It remains
+       attached to link6 and therefore does not rotate with rh_r1_joint. -->
+  <link name="$(arg prefix)teleop_task"/>
+  <joint name="$(arg prefix)teleop_task_fixed" type="fixed">
+    <parent link="$(arg prefix)link6"/>
+    <child link="$(arg prefix)teleop_task"/>
+    <origin xyz="0 -0.125 -0.0255" rpy="0 0 0"/>
+  </joint>
   <xacro:omy_l100_gazebo prefix="$(arg prefix)" />
   <xacro:omy_l100_system
